File: Nestick.sch (KiCad schematic (older format))
At the start: 16 parts, among them J1 CONN_EXT, J2 CONN_DIRS, J3 CONN_DGND, J4 CONN_BTNS, J5 CONN_BGND, Q1 2N3904, U1 74LS165, U2 74LS165

Commit message: Dress up for release
Parts:
- added H1, H2, H3, H4: HOLE, MountingHole:MountingHole_3.2mm_M3_Pad, symbol Mechanical:MountingHole_Pad
Connections:
- no-connect marks 3 -> 7
Other:
- moved on the sheet: J1, J2, J3, J4, J5
